Commit message: Add team colour setting, table frame and higher camera
- team_color launch argument (yellow|blue) on full_system and arena
  launches. robot_spawn.launch.py spawns the robot in that team's throne
  room and publishes table -> map at the start pose, so nodes and Nav2
  goals can use rule-book coordinates (frame_id: table).
- field.py: table layout from the rules (throne rooms, stables, quarries,
  stone size/ArUco id) with yellow/blue mirroring helpers.
- field_markers node draws the table in RViz. RViz now uses the table
  frame, centred on the table.
- Camera raised to ~0.33 m above the table and tilted 25 deg down, kept
  in sync in model.sdf, simple_robot.urdf and the perception parameters.
- teleop launch argument to run without the keyboard window.
- Robot spawns at its resting height.

Verified in sim for both colours: spawn pose matches Gazebo, table ->
base_link matches ground truth, and a Nav2 goal sent in the table frame
succeeds (within 2 mm of ground truth).

Co-Authored-By: Claude Opus 5.5 <noreply@anthropic.com>

File: src/mechaknights_2027/models/simple_robot/simple_robot.urdf (robot description, URDF)
Before this commit: robot simple_robot, 10 links, 9 joints
Joints:
- joint camera_joint: origin (none) -> xyz=0.10 0 0.29 rpy=0 0.436 0

Commit message: Add stone perception with 3D positions and an accuracy check
- stone_perception node: detects the stones' ArUco marker (ID 13, 80 mm)
  at several image scales (close-up markers were missed at full scale),
  estimates each marker pose, moves to the stone centre and reports it in
  the table frame through TF: x, y, z, yaw, stack level, top-face height
  (top_z, for grabbing from above) and whether it is the top of its stack.
  Publishes /stones/detections, a /stones/debug preview with the
  detections drawn, and /stones/markers for RViz. full_system now runs it
  instead of the 2026 crate detector.
- New StoneDetection / StoneDetectionArray messages.
- stone_accuracy tool (simulation only): compares detections with Gazebo
  ground truth and splits the error into camera, localisation and height.
- TF fix: odometry now moves base_footprint (on the table) with base_link
  40 mm above it, and SLAM uses base_footprint. Before, every height was
  40 mm low.

Measured in sim: camera error 1-2 mm at 0.6 m and ~10 mm at 1.4 m, height
error 0-1 mm, stack level always correct. Remaining error comes from
localisation after driving (4-8 cm, up to 6 deg).

Co-Authored-By: Claude Opus 5.5 <noreply@anthropic.com>

File: src/mechaknights_2027/models/simple_robot/simple_robot.urdf (robot description, URDF)
Before this commit: robot simple_robot, 10 links, 9 joints
Joints:
- joint base_to_footprint: child base_footprint -> base_link; origin (none) -> xyz=0 0 0.040 rpy=0 0 0; parent base_link -> base_footprint
